File: KiCAD_Project/learning_shield/learning_shield.sch (KiCad schematic (older format))
At the start: 43 parts, among them J1 Ping Sensor, J2 Servo, P1 Power, P2 Analog, P3 Digital, P4 Digital, P5 CONN_01X01, P6 CONN_01X01, P7 CONN_01X01, P8 CONN_01X01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

Commit message: Update part numbers and population status.
Parts:
- BZ1: Internal Part Number (none) -> 1-0000647
- C1, C2, C3, C4, J1, J2, P1, P2, P3, P4, P5, P6, P7, P8: Internal Part Number (none) -> 0-0000000; Populated (none) -> 0
- D1: Internal Part Number (none) -> 1-0000598; Populated (none) -> 1
- D2: value LED A -> LED B; Internal Part Number (none) -> 1-0000600; Populated (none) -> 1
- D3: value LED A -> LED C; Internal Part Number (none) -> 1-0000599; Populated (none) -> 1
- D4: value LED A -> LED D; Internal Part Number (none) -> 1-0000601; Populated (none) -> 1
- R9: Internal Part Number (none) -> 1-0000646; Populated (none) -> 1
- RV1: value R_POT -> 5k; Internal Part Number (none) -> 1-0000645; Populated (none) -> 0
- SW1, SW2, SW3, SW4: Internal Part Number (none) -> 1-0000643; Populated (none) -> 1
- U1: Internal Part Number (none) -> 1-0000259; Populated (none) -> 1
- U2: Internal Part Number (none) -> 1-0000644; Populated (none) -> 1
Other:
- note added: "Blue"
- note added: "Green"
- note added: "NP"
- note added: "Red"
- note added: "Yellow"

Commit message: Add final BOM/files
Parts:
- added PCB1: barepcb, symbol lib_fp:barepcb
Changed lines of the file:
@@
 Text Notes 3850 3125 0    50   ~ 0
 NP
+$Comp
+L lib_fp:barepcb PCB1
+U 1 1 5FDF0564
+P 7175 6350
+F 0 "PCB1" H 7403 6396 50  0000 L CNN
+F 1 "barepcb" H 7025 6375 50  0000 L CNN
+F 2 "" H 7175 6350 50  0001 C CNN
+F 3 "" H 7175 6350 50  0001 C CNN
+F 4 "3-0000025" H 7175 6350 50  0001 C CNN "Internal Part Number"
+F 5 "1" H 7175 6350 50  0001 C CNN "Populated"
+	1    7175 6350
+	1    0    0    -1
+$EndComp
 $EndSCHEMATC
